Commit message: feat: Add actuator and sensor plugins
Add camera, lidar, and differential drive plugins.

File: my_robot/urdf/my_robot.xacro (robot description, xacro)
@@ -1,4 +1,5 @@
 <?xml version="1.0"?>
 <robot name="my_robot" xmlns:xacro="http://www.ros.org.wiki/xacro">
+  <xacro:include filename="$(find my_robot)/urdf/my_robot.gazebo"/>
   <link name="robot_footprint"></link>
   <joint name="robot_footprint_joint" type="fixed">
@@ -10,5 +11,5 @@
     <pose>0 0 0.15 0 0 0</pose>
     <inertial>
-      <mass value="20.0"/>
+      <mass value="12.0"/>
       <origin xyz="0 0 0" rpy="0 0 0"/>
       <inertia
@@ -45,5 +46,5 @@
   <link name="left_wheel">
     <inertial>
-      <mass value="6.0"/>
+      <mass value="4.0"/>
       <origin xyz="0 0 0" rpy="0 1.5707 1.5707"/>
       <inertia
@@ -76,5 +77,5 @@
   <link name="right_wheel">
     <inertial>
-      <mass value="6.0"/>
+      <mass value="4.0"/>
       <origin xyz="0 0 0" rpy="0 1.5707 1.5707"/>
       <inertia
@@ -103,5 +104,63 @@
     <axis xyz="0 1 0" rpy="0 0 0"/>
     <limit effort="10000" velocity="1000"/>
-    <dynamics damping="1.0" friction="1.0"/>
+    <dynamics damping="1.0" friction="0.5"/>
+  </joint>
+  <link name="camera">
+    <inertial>
+      <mass value="1e-5"/>
+      <origin xyz="0 0 0" rpy="0 0 0"/>
+      <inertia
+        ixx="1e-6" ixy="0" ixz="0"
+        iyy="1e-6" iyz="0"
+        izz="1e-6"
+      />
+    </inertial>
+    <collision name="camera_collision">
+      <origin xyz="0 0 0" rpy="0 0 0"/>
+      <geometry>
+        <box size="0.05 0.05 0.05"/>
+      </geometry>
+    </collision>
+    <visual name="camera_visual">
+      <origin xyz="0 0 0" rpy="0 0 0"/>
+      <geometry>
+        <box size="0.05 0.05 0.05"/>
+      </geometry>
+    </visual>
+  </link>
+  <joint type="fixed" name="camera_joint">
+    <origin xyz="0.35 0 0" rpy="0 0 0"/>
+    <child link="camera"/>
+    <parent link="chassis"/>
+    <axis xyz="0 1 0" rpy="0 0 0"/>
+  </joint>
+  <link name="hokuyo">
+    <inertial>
+      <mass value="1e-5"/>
+      <origin xyz="0 0 0" rpy="0 0 0"/>
+      <inertia
+        ixx="1e-6" ixy="0" ixz="0"
+        iyy="1e-6" iyz="0"
+        izz="1e-6"
+      />
+    </inertial>
+    <collision name="hokuyo_collision">
+      <origin xyz="0 0 0" rpy="0 0 0"/>
+      <geometry>
+        <box size="0.1 0.1 0.1"/>
+      </geometry>
+    </collision>
+    <visual name="hokuyo_visual">
+      <origin xyz="0 0 0" rpy="0 0 0"/>
+      <geometry>
+        <mesh filename="package://my_robot/meshes/hokuyo.dae"/>
+      </geometry>
+    </visual>
+  </link>
+  <joint type="fixed" name="hokuyo_joint">
+    <origin xyz="0.3 0 0.1" rpy="0 0 0"/>
+    <child link="hokuyo"/>
+    <parent link="chassis"/>
+    <axis xyz="0 1 0" rpy="0 0 0"/>
   </joint>
 </robot>

Commit message: feat: Revert to original world with T-shaped robot
Revert to world from project 1, with a T-shaped robot with red
and blue wheels.

File: my_robot/urdf/my_robot.xacro (robot description, xacro)
@@ -1,16 +1,16 @@
 <?xml version="1.0"?>
-<robot name="my_robot" xmlns:xacro="http://www.ros.org.wiki/xacro">
-  <xacro:include filename="$(find my_robot)/urdf/my_robot.gazebo"/>
+<robot name="my_robot" xmlns:xacro="http://www.ros.org/wiki/xacro">
+  <xacro:include filename="$(find my_robot)/urdf/my_robot.gazebo" />
   <link name="robot_footprint"></link>
   <joint name="robot_footprint_joint" type="fixed">
-    <origin xyz="0 0 0" rpy="0 0 0"/>
-    <parent link="robot_footprint"/>
-    <child link="chassis"/>
+    <origin xyz="0 0 0" rpy="0 0 0" />
+    <parent link="robot_footprint" />
+    <child link="chassis" />
   </joint>
   <link name="chassis">
-    <pose>0 0 0.15 0 0 0</pose>
+    <pose>0 0 0.1 0 0 0</pose>
     <inertial>
-      <mass value="12.0"/>
-      <origin xyz="0 0 0" rpy="0 0 0"/>
+      <mass value="15.0" />
+      <origin xyz="0 0 0" rpy="0 0 0" />
       <inertia
         ixx="0.1" ixy="0" ixz="0"
@@ -19,26 +19,39 @@
       />
     </inertial>
-    <collision name="chassis_collision">
-      <origin xyz="0 0 0" rpy="0 0 0"/>
+    <collision name="chassis_front_collision">
+      <origin xyz="0 0 0" rpy="0 0 0" />
       <geometry>
-        <box size="0.7 0.4 0.1"/>
+        <box size=".2 .6 .1" />
       </geometry>
     </collision>
-    <visual name="chassis_visual">
-      <origin xyz="0 0 0" rpy="0 0 0"/>
+    <visual name="chassis_front_visual">
+      <origin xyz="0 0 0" rpy="0 0 0" />
       <geometry>
-        <box size="0.7 0.4 0.1"/>
+        <box size=".2 .6 .1" />
+      </geometry>
+      <material name="orange"/>
+    </visual>
+    <collision name="chassis_back_collision">
+      <origin xyz="-.3 0 0" rpy="0 0 0" />
+      <geometry>
+        <box size=".4 .2 .1" />
+      </geometry>
+    </collision>
+    <visual name="chassis_back_visual">
+      <origin xyz="-.3 0 0" rpy="0 0 0" />
+      <geometry>
+        <box size=".4 .2 .1" />
       </geometry>
     </visual>
     <collision name="back_caster_collision">
-      <origin xyz="-0.25 0 -0.05" rpy="0 0 0"/>
+      <origin xyz="-0.4 0 -0.05" rpy="0 0 0" />
       <geometry>
-        <sphere radius="0.1"/>
+        <sphere radius="0.05" />
       </geometry>
     </collision>
     <visual name="back_caster_visual">
-      <origin xyz="-0.25 0 -0.05" rpy="0 0 0"/>
+      <origin xyz="-0.4 0 -0.05" rpy="0 0 0" />
       <geometry>
-        <sphere radius="0.1"/>
+        <sphere radius="0.05" />
       </geometry>
     </visual>
@@ -46,68 +59,93 @@
   <link name="left_wheel">
     <inertial>
-      <mass value="4.0"/>
-      <origin xyz="0 0 0" rpy="0 1.5707 1.5707"/>
+      <mass value="5.0" />
+      <origin xyz="0 0 0" rpy="0 1.5707 1.5707" />
       <inertia
-        ixx="0.15" ixy="0" ixz="0"
-        iyy="0.15" iyz="0"
-        izz="0.15"
+        ixx="0.1" ixy="0" ixz="0"
+        iyy="0.1" iyz="0"
+        izz="0.1"
       />
     </inertial>
-    <collision name="left_wheel_collision">
-      <origin xyz="0 0 0" rpy="0 1.57 1.57"/>
+    <collision>
+      <origin xyz="0 0 0" rpy="0 1.5707 1.5707" />
       <geometry>
-        <cylinder radius="0.15" length="0.05"/>
+        <cylinder radius="0.1" length="0.05" />
       </geometry>
     </collision>
-    <visual name="left_wheel_visual">
-      <origin xyz="0 0 0" rpy="0 1.57 1.57"/>
+    <visual>
+      <origin xyz="0 0 0" rpy="0 1.5707 1.5707" />
       <geometry>
-        <cylinder radius="0.15" length="0.05"/>
+        <cylinder radius="0.1" length="0.05" />
       </geometry>
     </visual>
   </link>
-  <joint type="continuous" name="left_wheel_hinge">
-    <origin xyz="0.20858 0.225 0" rpy="0 0 0"/>
-    <child link="left_wheel"/>
-    <parent link="chassis"/>
-    <axis xyz="0 1 0" rpy="0 0 0"/>
-    <limit effort="10000" velocity="1000"/>
-    <dynamics damping="1.0" friction="1.0"/>
-  </joint>
   <link name="right_wheel">
     <inertial>
-      <mass value="4.0"/>
-      <origin xyz="0 0 0" rpy="0 1.5707 1.5707"/>
+      <mass value="5.0" />
+      <origin xyz="0 0 0" rpy="0 1.5707 1.5707" />
       <inertia
-        ixx="0.15" ixy="0" ixz="0"
-        iyy="0.15" iyz="0"
-        izz="0.15"
+        ixx="0.1" ixy="0" ixz="0"
+        iyy="0.1" iyz="0"
+        izz="0.1"
       />
     </inertial>
-    <collision name="right_wheel_collision">
-      <origin xyz="0 0 0" rpy="0 1.57 1.57"/>
+    <collision>
+      <origin xyz="0 0 0" rpy="0 1.5707 1.5707" />
       <geometry>
-        <cylinder radius="0.15" length="0.05"/>
+        <cylinder radius="0.1" length="0.05" />
       </geometry>
     </collision>
-    <visual name="right_wheel_visual">
-      <origin xyz="0 0 0" rpy="0 1.57 1.57"/>
+    <visual>
+      <origin xyz="0 0 0" rpy="0 1.5707 1.5707" />
       <geometry>
-        <cylinder radius="0.15" length="0.05"/>
+        <cylinder radius="0.1" length="0.05" />
       </geometry>
     </visual>
   </link>
+  <gazebo reference="left_wheel">
+    <material>Gazebo/Blue</material>
+  </gazebo>
+  <gazebo reference="right_wheel">
+    <material>Gazebo/Red</material>
+  </gazebo>
+  <joint type="continuous" name="left_wheel_hinge">
+    <origin xyz="0 0.325 0" rpy="0 0 0" />
+    <child link="left_wheel" />
+    <parent link="chassis" />
+    <axis xyz="0 1 0" rpy="0 0 0" />
+    <limit effort="10000" velocity="1000" />
+    <dynamics damping="1.0" friction="1.0" />
+  </joint>
   <joint type="continuous" name="right_wheel_hinge">
-    <origin xyz="0.20858 -0.225 0" rpy="0 0 0"/>
-    <child link="right_wheel"/>
-    <parent link="chassis"/>
-    <axis xyz="0 1 0" rpy="0 0 0"/>
-    <limit effort="10000" velocity="1000"/>
-    <dynamics damping="1.0" friction="0.5"/>
+    <origin xyz="0 -0.325 0" rpy="0 0 0" />
+    <child link="right_wheel" />
+    <parent link="chassis" />
+    <axis xyz="0 1 0" rpy="0 0 0" />
+    <limit effort="10000" velocity="1000" />
+    <dynamics damping="1.0" friction="1.0" />
   </joint>
   <link name="camera">
+    <box_inertia x="0.05" y="0.05" z="0.05" m="0.1" />
+    <collision>
+      <origin xyz="0 0 0" rpy="0 0 0" />
+      <geometry>
+        <box size="0.05 0.05 0.05" />
+      </geometry>
+    </collision>
+    <visual>
+      <origin xyz="0 0 0" rpy="0 0 0" />
+      <geometry>
+        <box size="0.05 0.05 0.05" />
+      </geometry>
+    </visual>
+  </link>
+  <joint type="fixed" name="camera_joint">
+    <origin xyz="0.1 0 0" rpy="0 0 0" />
+    <parent link="chassis" />
+    <child link="camera" />
+  </joint>
+  <link name="hokuyo">
     <inertial>
-      <mass value="1e-5"/>
-      <origin xyz="0 0 0" rpy="0 0 0"/>
+      <mass value="1e-5" />
       <inertia
         ixx="1e-6" ixy="0" ixz="0"
@@ -116,51 +154,21 @@
       />
     </inertial>
-    <collision name="camera_collision">
-      <origin xyz="0 0 0" rpy="0 0 0"/>
+    <collision>
+      <origin xyz="0 0 0" rpy="0 0 0" />
       <geometry>
-        <box size="0.05 0.05 0.05"/>
+        <box size="0.1 0.1 0.1" />
       </geometry>
     </collision>
-    <visual name="camera_visual">
-      <origin xyz="0 0 0" rpy="0 0 0"/>
+    <visual>
+      <origin xyz="0 0 0" rpy="0 0 0" />
       <geometry>
-        <box size="0.05 0.05 0.05"/>
+        <mesh filename="package://my_robot/meshes/hokuyo.dae" />
       </geometry>
     </visual>
   </link>
-  <joint type="fixed" name="camera_joint">
-    <origin xyz="0.35 0 0" rpy="0 0 0"/>
-    <child link="camera"/>
-    <parent link="chassis"/>
-    <axis xyz="0 1 0" rpy="0 0 0"/>
-  </joint>
-  <link name="hokuyo">
-    <inertial>
-      <mass value="1e-5"/>
-      <origin xyz="0 0 0" rpy="0 0 0"/>
-      <inertia
-        ixx="1e-6" ixy="0" ixz="0"
-        iyy="1e-6" iyz="0"
-        izz="1e-6"
-      />
-    </inertial>
-    <collision name="hokuyo_collision">
-      <origin xyz="0 0 0" rpy="0 0 0"/>
-      <geometry>
-        <box size="0.1 0.1 0.1"/>
-      </geometry>
-    </collision>
-    <visual name="hokuyo_visual">
-      <origin xyz="0 0 0" rpy="0 0 0"/>
-      <geometry>
-        <mesh filename="package://my_robot/meshes/hokuyo.dae"/>
-      </geometry>
-    </visual>
-  </link>
-  <joint type="fixed" name="hokuyo_joint">
-    <origin xyz="0.3 0 0.1" rpy="0 0 0"/>
-    <child link="hokuyo"/>
-    <parent link="chassis"/>
-    <axis xyz="0 1 0" rpy="0 0 0"/>
+  <joint name="hokuyo" type="fixed">
+    <origin xyz="0.05 0 0.1" rpy="0 0 0"/>
+    <parent link="chassis" />
+    <child link="hokuyo" />
   </joint>
 </robot>

Commit message: feat: Make robot chase white ball
Make the robot chase the white ball based on where in the camera
image the ball is located.

File: my_robot/urdf/my_robot.xacro (robot description, xacro)
@@ -8,5 +8,5 @@
     <child link="chassis" />
   </joint>
-  <link name="chassis">
+  <link name="chassis_front">
     <pose>0 0 0.1 0 0 0</pose>
     <inertial>
@@ -44,4 +44,15 @@
       </geometry>
     </visual>
+  </link>
+  <link name="back_caster">
+    <inertial>
+      <mass value="10.0" />
+      <origin xyz="0 0 0" rpy="0 0 0" />
+      <inertia
+        ixx="0.1" ixy="0" ixz="0"
+        iyy="0.1" iyz="0"
+        izz="0.1"
+      />
+    </inertial>
     <collision name="back_caster_collision">
       <origin xyz="-0.4 0 -0.05" rpy="0 0 0" />
@@ -57,4 +68,9 @@
     </visual>
   </link>
+  <joint type="fixed" name="back_caster_hinge">
+    <origin xyz="-0.4 0 -0.05" rpy="0 0 0" />
+    <child link="back_caster" />
+    <parent link="chassis" />
+  </joint>
   <link name="left_wheel">
     <inertial>

Commit message: fix: Fix my_robot definition
Fix errors in my_robot.xacro file

File: my_robot/urdf/my_robot.xacro (robot description, xacro)
@@ -8,5 +8,5 @@
     <child link="chassis" />
   </joint>
-  <link name="chassis_front">
+  <link name="chassis">
     <pose>0 0 0.1 0 0 0</pose>
     <inertial>

Commit message: fix: Fix world file so there isn't already a robot
Save the world file so there isn't a robot in there already when launching
the world.launch file.

File: my_robot/urdf/my_robot.xacro (robot description, xacro)
@@ -19,5 +19,17 @@
       />
     </inertial>
-    <collision name="chassis_front_collision">
+    <collision name="chassis_collision_1">
+      <origin xyz="-.2 0 0" rpy="0 0 0" />
+      <geometry>
+        <box size="1.0 .2 .1" />
+      </geometry>
+    </collision>
+    <visual name="chassis_visual_1">
+      <origin xyz="-.2 0 0" rpy="0 0 0" />
+      <geometry>
+        <box size="1.0 .2 .1" />
+      </geometry>
+    </visual>
+    <collision name="chassis_collision_2">
       <origin xyz="0 0 0" rpy="0 0 0" />
       <geometry>
@@ -25,52 +37,35 @@
       </geometry>
     </collision>
-    <visual name="chassis_front_visual">
+    <visual name="chassis_visual_2">
       <origin xyz="0 0 0" rpy="0 0 0" />
       <geometry>
         <box size=".2 .6 .1" />
       </geometry>
-      <material name="orange"/>
     </visual>
-    <collision name="chassis_back_collision">
-      <origin xyz="-.3 0 0" rpy="0 0 0" />
+    <collision name="back_caster_collision">
+      <origin xyz="-0.65 0 -0.05" rpy="0 0 0" />
       <geometry>
-        <box size=".4 .2 .1" />
+        <sphere radius="0.0499" />
       </geometry>
     </collision>
-    <visual name="chassis_back_visual">
-      <origin xyz="-.3 0 0" rpy="0 0 0" />
+    <visual name="back_caster_visual">
+      <origin xyz="-0.65 0 -0.05" rpy="0 0 0" />
       <geometry>
-        <box size=".4 .2 .1" />
+        <sphere radius="0.0499" />
+      </geometry>
+    </visual>
+    <collision name="front_caster_collision">
+      <origin xyz="0.25 0 -0.05" rpy="0 0 0" />
+      <geometry>
+        <sphere radius="0.0499" />
+      </geometry>
+    </collision>
+    <visual name="front_caster_visual">
+      <origin xyz="0.25 0 -0.05" rpy="0 0 0" />
+      <geometry>
+        <sphere radius="0.0499" />
       </geometry>
     </visual>
   </link>
-  <link name="back_caster">
-    <inertial>
-      <mass value="10.0" />
-      <origin xyz="0 0 0" rpy="0 0 0" />
-      <inertia
-        ixx="0.1" ixy="0" ixz="0"
-        iyy="0.1" iyz="0"
-        izz="0.1"
-      />
-    </inertial>
-    <collision name="back_caster_collision">
-      <origin xyz="-0.4 0 -0.05" rpy="0 0 0" />
-      <geometry>
-        <sphere radius="0.05" />
-      </geometry>
-    </collision>
-    <visual name="back_caster_visual">
-      <origin xyz="-0.4 0 -0.05" rpy="0 0 0" />
-      <geometry>
-        <sphere radius="0.05" />
-      </geometry>
-    </visual>
-  </link>
-  <joint type="fixed" name="back_caster_hinge">
-    <origin xyz="-0.4 0 -0.05" rpy="0 0 0" />
-    <child link="back_caster" />
-    <parent link="chassis" />
-  </joint>
   <link name="left_wheel">
     <inertial>
@@ -156,6 +151,9 @@
     </visual>
   </link>
+  <gazebo reference="camera">
+    <material>Gazebo/Green</material>
+  </gazebo>
   <joint type="fixed" name="camera_joint">
-    <origin xyz="0.1 0 0" rpy="0 0 0" />
+    <origin xyz="0.3 0 0" rpy="0 0 0" />
     <parent link="chassis" />
     <child link="camera" />
@@ -184,5 +182,5 @@
   </link>
   <joint name="hokuyo" type="fixed">
-    <origin xyz="0.05 0 0.1" rpy="0 0 0"/>
+    <origin xyz="0.25 0 0.08" rpy="0 0 0"/>
     <parent link="chassis" />
     <child link="hokuyo" />
